File: Kicad_Files/Trugbild.kicad_pcb (KiCad board)
At the start: 4 copper layers, 85 x 40 mm, 97 parts, among them J1 Conn_02x05_Odd_Even, J2 HDMI_A, J3 Conn_01x02, J4 HDMI_A, U1 AS4C32M8SA-6TIN, U2 XC3S50A-4VQG100C, U3 MIC5365-3.3YD5, U4 LDK130PU12R_DFN6, U5 MX25L1636EM2I-08G, X1 EC5645ETTS-50.000M

Commit message: fix for clearance v2
Parts:
- moved C35 0.13 mm to (166.6, 103.6)
Routing:
- net /SCL_IN: track 40.7 -> 39.5 mm
- net /UTIL_IN: track 40.4 -> 39.2 mm
Other:
- net class Matched: clearance 0.09 -> 0.1; trace_width 0.09 -> 0.1
- rule trace_min: 0.0889 -> 0.1
- rule via_min_size: 0.45 -> 0.2
